File: KICAD/CPU_Power_Supply_Mod/CPU_Power_Supply_Mod.kicad_pcb (KiCad board)
At the start: 2 copper layers, 37 parts, among them K1 RELAY_SPST, K2 RELAY_SPST, K3 RELAY_SPST, K4 RELAY_SPST, P1 CONN_6, P2 CONN-12X2, P3 CONN_6, P4 CONN_2X2, Q1 PN2907, Q2 PN2907, Q3 PN2907, Q4 PN2907, SW1 SW_PUSH, SW2 SW_PUSH, SW3 SW_PUSH, U1 PIC18F1220, U2 74HC595N, U3 16X2_LCD

Commit message: Updated PCB
Parts:
- F1, F2, F3: value FUSE -> 2.5A
- P1: value CONN_6 -> ICSP
- P2: value CONN-12X2 -> ATX 2.x
- P3: value CONN_6 -> PWR OUT
- P4: value CONN_2X2 -> PG SWT
- SW1, SW2, SW3: value SW_PUSH -> (none)
Routing:
- added copper zone on F.Cu, net N-0000048
- removed copper zone on F.Cu, net N-0000047

Commit message: Updated Schematic
Changed lines of the file:
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@@
   (module SW_PUSH_SMALL (layer F.Cu)
     (at 97.05 149.2 180)
-    (fp_text reference SW3 (at 0 -0.762 180) (layer F.SilkS)
+    (fp_text reference SW3 (at 5.8 -0.3 180) (layer F.SilkS)
       (effects (font (size 1.016 1.016) (thickness 0.2032)))
     )
@@
   (module SW_PUSH_SMALL (layer F.Cu)
     (at 75.4 149.2 180)
-    (fp_text reference SW2 (at 0 -0.762 180) (layer F.SilkS)
+    (fp_text reference SW2 (at 5.65 -0.05 180) (layer F.SilkS)
       (effects (font (size 1.016 1.016) (thickness 0.2032)))
     )
@@
   (module SW_PUSH_SMALL (layer F.Cu)
     (at 52.2 149.25 180)
-    (fp_text reference SW1 (at 0 -0.762 180) (layer F.SilkS)
+    (fp_text reference SW1 (at 5.7 0 180) (layer F.SilkS)
       (effects (font (size 1.016 1.016) (thickness 0.2032)))
     )
@@
     (tags R)
     (autoplace_cost180 10)
-    (fp_text reference R4 (at 6.2 -0.15 180) (layer F.SilkS) hide
-      (effects (font (size 1.397 1.27) (thickness 0.2032)))
-    )
-    (fp_text value R (at 0 0.127 180) (layer F.SilkS)
+    (fp_text reference R4 (at 6.2 -0.15 180) (layer F.SilkS)
+      (effects (font (size 1.397 1.27) (thickness 0.2032)))
+    )
+    (fp_text value R (at 0 0.127 180) (layer F.SilkS) hide
       (effects (font (size 1.397 1.27) (thickness 0.2032)))
     )
@@
     (tags R)
     (autoplace_cost180 10)
-    (fp_text reference R7 (at -6.05 0.1) (layer F.SilkS) hide
-      (effects (font (size 1.397 1.27) (thickness 0.2032)))
-    )
-    (fp_text value R (at 0 0.127) (layer F.SilkS)
+    (fp_text reference R7 (at -6.05 0.1) (layer F.SilkS)
+      (effects (font (size 1.397 1.27) (thickness 0.2032)))
+    )
+    (fp_text value R (at 0 0.127) (layer F.SilkS) hide
       (effects (font (size 1.397 1.27) (thickness 0.2032)))
     )
@@
     (tags R)
     (autoplace_cost180 10)
-    (fp_text reference R3 (at 6.3 -0.15 180) (layer F.SilkS) hide
-      (effects (font (size 1.397 1.27) (thickness 0.2032)))
-    )
-    (fp_text value R (at 0 0.127 180) (layer F.SilkS)
+    (fp_text reference R3 (at 6.3 -0.15 180) (layer F.SilkS)
+      (effects (font (size 1.397 1.27) (thickness 0.2032)))
+    )
+    (fp_text value R (at 0 0.127 180) (layer F.SilkS) hide
       (effects (font (size 1.397 1.27) (thickness 0.2032)))
     )
@@
     (tags R)
     (autoplace_cost180 10)
-    (fp_text reference R2 (at -6.3 -0.2 90) (layer F.SilkS) hide
-      (effects (font (size 1.397 1.27) (thickness 0.2032)))
-    )
-    (fp_text value R (at 0 0.127 90) (layer F.SilkS)
+    (fp_text reference R2 (at -6.3 -0.2 90) (layer F.SilkS)
+      (effects (font (size 1.397 1.27) (thickness 0.2032)))
+    )
+    (fp_text value R (at 0 0.127 90) (layer F.SilkS) hide
       (effects (font (size 1.397 1.27) (thickness 0.2032)))
     )
@@
     (tags R)
     (autoplace_cost180 10)
-    (fp_text reference R1 (at -6.3 0.1 90) (layer F.SilkS) hide
-      (effects (font (size 1.397 1.27) (thickness 0.2032)))
-    )
-    (fp_text value R (at 0 0.127 90) (layer F.SilkS)
+    (fp_text reference R1 (at -6.3 0.1 90) (layer F.SilkS)
+      (effects (font (size 1.397 1.27) (thickness 0.2032)))
+    )
+    (fp_text value R (at 0 0.127 90) (layer F.SilkS) hide
       (effects (font (size 1.397 1.27) (thickness 0.2032)))
     )
@@
     (tags R)
     (autoplace_cost180 10)
-    (fp_text reference R5 (at -6.3 0.2) (layer F.SilkS) hide
-      (effects (font (size 1.397 1.27) (thickness 0.2032)))
-    )
-    (fp_text value R (at 0 0.127) (layer F.SilkS)
+    (fp_text reference R5 (at -6.05 0.2) (layer F.SilkS)
+      (effects (font (size 1.397 1.27) (thickness 0.2032)))
+    )
+    (fp_text value R (at 0 0.127) (layer F.SilkS) hide
       (effects (font (size 1.397 1.27) (thickness 0.2032)))
     )
@@
     (tags R)
     (autoplace_cost180 10)
-    (fp_text reference R6 (at 6.4 -0.2 180) (layer F.SilkS) hide
-      (effects (font (size 1.397 1.27) (thickness 0.2032)))
-    )
-    (fp_text value R (at 0 0.127 180) (layer F.SilkS)
+    (fp_text reference R6 (at 6.15 -0.2 180) (layer F.SilkS)
+      (effects (font (size 1.397 1.27) (thickness 0.2032)))
+    )
+    (fp_text value R (at -0.1 0.05 180) (layer F.SilkS) hide
       (effects (font (size 1.397 1.27) (thickness 0.2032)))
     )
@@
     (at 63.35 134.35)
     (descr "8 pins DIL package, round pads")
-    (fp_text reference U1 (at -7.62 -1.27) (layer F.SilkS)
+    (fp_text reference U1 (at -14.1 0.15 90) (layer F.SilkS)
       (effects (font (size 1.778 1.143) (thickness 0.3048)))
     )
-    (fp_text value PIC18F1220 (at 5.08 1.27) (layer F.SilkS)
+    (fp_text value PIC18F1220 (at -2.35 0.4) (layer F.SilkS)
       (effects (font (size 1.778 1.143) (thickness 0.3048)))
     )
@@
     (descr "16 pins DIL package, round pads")
     (tags DIL)
-    (fp_text reference U2 (at -6.35 -1.27 180) (layer F.SilkS)
+    (fp_text reference U2 (at 12.85 0.1 270) (layer F.SilkS)
       (effects (font (size 1.524 1.143) (thickness 0.3048)))
     )
-    (fp_text value 74HC595N (at 2.54 1.27 180) (layer F.SilkS)
+    (fp_text value 74HC595N (at 2.85 -0.15 180) (layer F.SilkS)
       (effects (font (size 1.524 1.143) (thickness 0.3048)))
     )
@@
   (module CON_3x1 (layer F.Cu)
     (at 41.55 116.35 270)
-    (fp_text reference RV1 (at -7.874 -2.286 270) (layer F.SilkS)
+    (fp_text reference RV1 (at -7.85 -2.45 270) (layer F.SilkS)
       (effects (font (size 1 1) (thickness 0.15)))
     )
-    (fp_text value POT (at -2.794 -2.286 270) (layer F.SilkS)
+    (fp_text value POT (at -2.85 -2.45 270) (layer F.SilkS)
       (effects (font (size 1 1) (thickness 0.15)))
     )
@@
     (descr "Condensateur e = 1 pas")
     (tags C)
-    (fp_text reference C3 (at 2.3 -2.25 270) (layer F.SilkS)
+    (fp_text reference C3 (at -0.2 -2.25 270) (layer F.SilkS)
       (effects (font (size 1.016 1.016) (thickness 0.2032)))
     )
@@
     (descr "Condensateur e = 1 pas")
     (tags C)
-    (fp_text reference C2 (at 2.45 -2.3 180) (layer F.SilkS)
+    (fp_text reference C2 (at 0.2 -2.3 180) (layer F.SilkS)
       (effects (font (size 1.016 1.016) (thickness 0.2032)))
     )
@@
     (descr "Condensateur e = 1 pas")
     (tags C)
-    (fp_text reference C1 (at -2.85 -2.1) (layer F.SilkS)
-      (effects (font (size 1.016 1.016) (thickness 0.2032)))
-    )
+    (fp_text reference C1 (at 0.15 -2.1) (layer F.SilkS)
+      (effects (font (size 1.016 1.016) (thickness 0.2032)))
+    )

Commit message: Finished Project
Parts:
- added R8: 10K, R3, F.Cu at (43.2, 136.0)
- SW1, SW2, SW3: value (none) -> SW_PUSH
Routing:
- net +5VA: track 425.3 -> 428.4 mm
- added copper zone on F.Cu, net N-0000048
- removed copper zone on F.Cu, net N-0000041
