File: KICAD/CPU_Power_Supply_Mod/CPU_Power_Supply_Mod.sch (KiCad schematic (older format))
At the start: 37 parts, among them K1 RELAY_SPST, K2 RELAY_SPST, K3 RELAY_SPST, K4 RELAY_SPST, P1 ICSP, P2 ATX 2.x, P3 PWR OUT, P4 PG SWT, Q1 PN2907, Q2 PN2907, Q3 PN2907, Q4 PN2907, SW1 SW_PUSH, SW2 SW_PUSH, SW3 SW_PUSH, U1 PIC18F1220, U2 74HC595N, U3 16X2_LCD

Commit message: Updated Schematic
Parts:
- added R?: 10K, ~, symbol R
Connections:
- net +5VA: now also R?.1
- net at P1.1, U1.4 (MCLR/VPP/RA5): now also R?.2
Changed lines of the file:
@@
 Sheet 1 1
 Title "CPU Power Supply Mod "
-Date "21 sep 2015"
+Date "29 oct 2015"
 Rev "1.0"
 Comp ""
@@
 	7350 2800 6950 2800
 Wire Wire Line
-	6950 2600 6950 2400
+	6950 2350 6950 2600
 Wire Wire Line
 	6950 2400 7350 2400
@@
 Wire Wire Line
 	6000 5750 5700 5750
+$Comp
+L R R?
+U 1 1 563288E8
+P 6950 2100
+F 0 "R?" V 7030 2100 40  0000 C CNN
+F 1 "10K" V 6957 2101 40  0000 C CNN
+F 2 "~" V 6880 2100 30  0000 C CNN
+F 3 "~" H 6950 2100 30  0000 C CNN
+	1    6950 2100
+	1    0    0    -1
+$EndComp
+Connection ~ 6950 2400
+$Comp
+L +5VA #PWR?
+U 1 1 563289B3
+P 6950 1800
+F 0 "#PWR?" H 6950 1930 20  0001 C CNN
+F 1 "+5VA" H 6950 1900 30  0000 C CNN
+F 2 "" H 6950 1800 60  0000 C CNN
+F 3 "" H 6950 1800 60  0000 C CNN
+	1    6950 1800
+	1    0    0    -1
+$EndComp
+Wire Wire Line
+	6950 1800 6950 1850
 $EndSCHEMATC

Commit message: Finished Project
Parts:
- gave numbers to parts that had none: 1
Changed lines of the file:
@@
 Sheet 1 1
 Title "CPU Power Supply Mod "
-Date "29 oct 2015"
+Date "14 nov 2015"
 Rev "1.0"
 Comp ""
@@
 	6000 5750 5700 5750
 $Comp
-L R R?
+L R R8
 U 1 1 563288E8
 P 6950 2100
-F 0 "R?" V 7030 2100 40  0000 C CNN
+F 0 "R8" V 7030 2100 40  0000 C CNN
 F 1 "10K" V 6957 2101 40  0000 C CNN
 F 2 "~" V 6880 2100 30  0000 C CNN
@@
 Connection ~ 6950 2400
 $Comp
-L +5VA #PWR?
+L +5VA #PWR043
 U 1 1 563289B3
 P 6950 1800
-F 0 "#PWR?" H 6950 1930 20  0001 C CNN
+F 0 "#PWR043" H 6950 1930 20  0001 C CNN
 F 1 "+5VA" H 6950 1900 30  0000 C CNN
 F 2 "" H 6950 1800 60  0000 C CNN
